Commit message: add mamual grasp demo

File: urdf/robotiq_85_gripper_simple.urdf (robot description, URDF)
Before this commit: robot robotiq_85_gripper, 16 links, 15 joints
Links:
- removed link x_control
- added link base_link, mass 0
- link dummy_center_indicator_link: geometry visual box size=0.020 0.085 0.002
- link roll_control: mass 0 -> 1
Joints:
- joint center_x: limit lower=-0.5 upper=0.5 effort=1000.0 velocity=0.5 -> lower=-0.5 upper=0.5 effort=1000.0 velocity=0.02; parent x_control -> base_link
- joint center_y: limit lower=-0.5 upper=0.5 effort=1000.0 velocity=0.5 -> lower=-0.5 upper=0.5 effort=1000.0 velocity=0.02
- joint center_z: child roll_control -> yaw_control; limit lower=0 upper=1 effort=1000.0 velocity=0.5 -> lower=-0.5 upper=0.5 effort=1000.0 velocity=0.02
- joint gripper_pitch: child yaw_control -> roll_control; limit lower=-3.14 upper=3.14 effort=1000 velocity=100.0 -> lower=0 upper=3.14 effort=1000 velocity=3.14; origin (none) -> xyz=0.010 0 0
- joint gripper_roll: child pitch_control -> dummy_center_indicator_link; limit lower=-3.14 upper=3.14 effort=1000 velocity=100.0 -> lower=0 upper=3.14 effort=100000 velocity=3.14; origin (none) -> xyz=0.140 0 0
- joint gripper_yaw: child dummy_center_indicator_link -> pitch_control; limit lower=-3.14 upper=3.14 effort=1000 velocity=100.0 -> lower=-3.14 upper=3.14 effort=1000 velocity=3.14; origin (none) -> xyz=0.010 0 0
- joint robotiq_85_left_finger_tip_joint: limit lower=-3.14 upper=3.14 effort=0.1 velocity=100.0 -> lower=-3.14 upper=3.14 effort=0.1 velocity=3.14
- joint robotiq_85_left_inner_knuckle_joint: limit lower=-3.14 upper=3.14 effort=0.1 velocity=100.0 -> lower=-3.14 upper=3.14 effort=0.1 velocity=3.14
- joint robotiq_85_left_knuckle_joint: limit lower=0.0 upper=0.80285 effort=1000 velocity=0.5 -> lower=0.0 upper=0.80285 effort=1000 velocity=3.14
- joint robotiq_85_right_finger_tip_joint: limit lower=-3.14 upper=3.14 effort=0.1 velocity=100.0 -> lower=-3.14 upper=3.14 effort=0.1 velocity=3.14
- joint robotiq_85_right_inner_knuckle_joint: limit lower=-3.14 upper=3.14 effort=0.1 velocity=100.0 -> lower=-3.14 upper=3.14 effort=0.1 velocity=3.14
- joint robotiq_85_right_knuckle_joint: limit lower=-3.14 upper=3.14 effort=1000 velocity=100.0 -> lower=-3.14 upper=3.14 effort=1000 velocity=3.14

Commit message: add InverseKinematics calculation

File: urdf/robotiq_85_gripper_simple.urdf (robot description, URDF)
Before this commit: robot robotiq_85_gripper, 16 links, 15 joints
Links:
- link dummy_center_indicator_link: mass 0 -> 0.1
- link pitch_control: mass 0 -> 0.1
- link roll_control: mass 1 -> 0.1
- link y_control: mass 0 -> 0.1
- link yaw_control: mass 0 -> 0.1
- link z_control: mass 0 -> 0.1
Joints:
- joint center_x: limit lower=-0.5 upper=0.5 effort=1000.0 velocity=0.02 -> lower=-0.5 upper=0.5 effort=1000.0 velocity=0.2
- joint center_y: limit lower=-0.5 upper=0.5 effort=1000.0 velocity=0.02 -> lower=-0.5 upper=0.5 effort=1000.0 velocity=0.2
- joint center_z: limit lower=-0.5 upper=0.5 effort=1000.0 velocity=0.02 -> lower=-0.25 upper=1 effort=1000.0 velocity=0.2
- joint gripper_pitch: limit lower=0 upper=3.14 effort=1000 velocity=3.14 -> lower=-31.4 upper=31.4 effort=10000 velocity=3.14; origin xyz=0.010 0 0 -> (none)
- joint gripper_roll: limit lower=0 upper=3.14 effort=100000 velocity=3.14 -> lower=-31.4 upper=31.4 effort=100000 velocity=3.14; origin xyz=0.140 0 0 -> (none)
- joint gripper_yaw: limit lower=-3.14 upper=3.14 effort=1000 velocity=3.14 -> lower=-31.4 upper=31.4 effort=10000 velocity=3.14; origin xyz=0.010 0 0 -> (none)
